File: Hardware/LEDCUBE_VER0.kicad_pcb (KiCad board)
At the start: 2 copper layers, 73 x 60 mm, 32 parts, among them J1 Conn_01x02_Pin, Q1 IRF9540N, Q2 IRF9540N, Q3 IRF9540N, U2 TXS0108EPW, U3 MBI5026

Commit message: update power part ver 0
Parts:
- added D16: D_Schottky, Diode_SMD:D_2114_3652Metric_Pad1.85x3.75mm_HandSolder, F.Cu at (119.1, 101.9)
- added D17: LED, Diode_SMD:D_0805_2012Metric_Pad1.15x1.40mm_HandSolder, F.Cu at (119.1, 97.0)
- added R8: 500, Diode_SMD:D_0805_2012Metric_Pad1.15x1.40mm_HandSolder, F.Cu at (121.7, 97.0)
- J1: footprint TerminalBlock_Phoenix:TerminalBlock_Phoenix_MPT-0,5-2-2.54_1x02_P2.54mm_Horizontal -> TerminalBlock_Phoenix:TerminalBlock_Phoenix_PT-1,5-2-5.0-H_1x02_P5.00mm_Horizontal
- R1, R3, R5: value R -> 20
- R2, R4, R6: value R -> 300
- R7: value R -> 1K1
- moved J1 3.43 mm to (128.1, 101.8)
Connections:
- J1 pad 1: +5V -> Net-(D16-A)
- U1 pad 18: unconnected-(U1-3V3-Pad18) -> +3.3V
- U1 pad 19: unconnected-(U1-G-Pad19) -> GND
Routing:
- net +3.3V: track 54.1 -> 80.7 mm
- net +5V: track 206.2 -> 195.2 mm
- net Net-(D16-A): track 0.00 -> 6.76 mm
- net GND: track 152.8 -> 157.4 mm
- net Net-(D17-K): track 0.00 -> 2.54 mm

Commit message: update power part of ver 0
Parts:
- removed D16: D_Schottky, Diode_SMD:D_2114_3652Metric_Pad1.85x3.75mm_HandSolder
- added Q4: IRF9540N, Package_TO_SOT_THT:TO-220-3_Vertical, F.Cu at (120.7, 102.6)
- added R9: 10K, Diode_SMD:D_0805_2012Metric_Pad1.15x1.40mm_HandSolder, F.Cu at (122.2, 98.6)
- moved D17 2.34 mm to (117.3, 98.6), turned to 90 degrees
- moved R8 2.34 mm to (119.9, 98.6), turned to 90 degrees
- moved J1 1.27 mm to (128.1, 103.1)
Connections:
- U1 pad 39: unconnected-(U1-G-Pad39) -> GND
Routing:
- net GND: track 157.4 -> 209.7 mm
- net Net-(J1-Pin_1): track 6.76 -> 12.4 mm
- net Net-(Q4-G): track 0.00 -> 3.67 mm
- net +5V: track 195.2 -> 193.7 mm
