File: Hardware/LEDCUBE_VER0.kicad_sch (KiCad schematic)
At the start: 31 parts, among them Q1 IRF9540N, Q2 IRF9540N, Q3 IRF9540N, U2 TXS0108EPW, U3 MBI5026

Commit message: update sche test board
Parts:
- added J1: Conn_01x02_Pin, TerminalBlock_Phoenix:TerminalBlock_Phoenix_MPT-0,5-2-2.54_1x02_P2.54mm_Horizontal, symbol Connector:Conn_01x02_Pin
- C1, C2: footprint (none) -> Capacitor_SMD:C_0603_1608Metric_Pad1.08x0.95mm_HandSolder
- C3: footprint (none) -> Capacitor_SMD:C_0805_2012Metric_Pad1.18x1.45mm_HandSolder
- D1, D10, D11, D12, D13, D14, D15, D2, D3, D4, D5, D6, D7, D8, D9: footprint (none) -> LED_THT:LED_D5.0mm-4_RGB
- R1, R2, R3, R4, R5, R6, R7: footprint (none) -> Resistor_SMD:R_0805_2012Metric_Pad1.20x1.40mm_HandSolder
- U1: footprint (none) -> Tduyen_Library:STM32F1_BluePill
- U3: footprint (none) -> Tduyen_Library:SOP-24
Connections:
- net +5V: now also J1.1 (Pin_1)
- net B0: now also U3.7 (~{OUT2}); no longer U3.15 (~{OUT10})
- net B1: now also U3.10 (~{OUT5}); no longer U3.16 (~{OUT11})
- net B2: now also U3.13 (~{OUT8}); no longer U3.17 (~{OUT12})
- net B3: now also U3.16 (~{OUT11}); no longer U3.18 (~{OUT13})
- net G0: now also U3.6 (~{OUT1}); no longer U3.10 (~{OUT5})
- net G1: now also U3.9 (~{OUT4}); no longer U3.11 (~{OUT6})
- net G3: now also U3.15 (~{OUT10}); no longer U3.13 (~{OUT8})
- net G4: now also U3.18 (~{OUT13}); no longer U3.14 (~{OUT9})
- net GND: now also J1.2 (Pin_2)
- net R1: now also U3.8 (~{OUT3}); no longer U3.6 (~{OUT1})
- net R2: now also U3.11 (~{OUT6}); no longer U3.7 (~{OUT2})
- net R3: now also U3.14 (~{OUT9}); no longer U3.8 (~{OUT3})
- net R4: now also U3.17 (~{OUT12}); no longer U3.9 (~{OUT4})

Commit message: update power part ver 0
Parts:
- added D16: D_Schottky, Diode_SMD:D_2114_3652Metric_Pad1.85x3.75mm_HandSolder, symbol Device:D_Schottky
- added D17: LED, Diode_SMD:D_0805_2012Metric_Pad1.15x1.40mm_HandSolder, symbol Device:LED
- added R8: 500, Diode_SMD:D_0805_2012Metric_Pad1.15x1.40mm_HandSolder, symbol Device:R
- J1: footprint TerminalBlock_Phoenix:TerminalBlock_Phoenix_MPT-0,5-2-2.54_1x02_P2.54mm_Horizontal -> TerminalBlock_Phoenix:TerminalBlock_Phoenix_PT-1,5-2-5.0-H_1x02_P5.00mm_Horizontal
- R1, R3, R5: value R -> 20
- R2, R4, R6: value R -> 300
- R7: value R -> 1K1
Connections:
- net +3.3V: now also U1.18 (3V3)
- net +5V: now also D16.1 (K), D17.2 (A); no longer J1.1 (Pin_1)
- net GND: now also U1.19 (G), R8.2
- new net: D17.1 (K), R8.1
- new net: D16.2 (A), J1.1 (Pin_1)
- no-connect marks 40 -> 38
Other:
- moved on the sheet: C1, C2, C3, J1, R7

Commit message: update power part of ver 0
Parts:
- removed D16: D_Schottky, Diode_SMD:D_2114_3652Metric_Pad1.85x3.75mm_HandSolder, symbol Device:D_Schottky
- added Q4: IRF9540N, Package_TO_SOT_THT:TO-220-3_Vertical, symbol Transistor_FET:IRF9540N
- added R9: 10K, Diode_SMD:D_0805_2012Metric_Pad1.15x1.40mm_HandSolder, symbol Device:R
Connections:
- net +5V: now also Q4.3 (S)
- net GND: now also U1.39 (G), R9.2
- net at J1.1 (Pin_1): now also Q4.2 (D)
- new net: Q4.1 (G), R9.1
- no-connect marks 38 -> 37
Other:
- moved on the sheet: J1
